File: MotorShield.brd (EAGLE design)
At the start: 88.9 x 71.1 mm, 141 parts, among them IC3 MIC4607, Q1 DMT4002LPS, Q2 DMT4002LPS, Q3 DMT4002LPS, Q4 DMT4002LPS, Q5 DMT4002LPS, Q6 DMT4002LPS, Q7 BC847BS, Q8 BC847BS

Commit message: REVB version update
Parts:
- removed 1790: MCP1790-3302E/DB, Microchip_By_element14_Batch_1:SOT230P700X180-4N
- removed 5233: MIC5233, MIC5233:MIC5233_SOT_23
- removed C10, C11, C9: 100p, rcl:C0805
- removed C23: 1u 50V, rcl:C0805
- removed C30: 100n, rcl:C0805
- removed DC_BUS_TP, P_CUR_1_TP, P_CUR_2_TP, P_CUR_SUM_TP: (no value), pinhead:1X01
- removed IC3: MIC4607, daniic:TSSOP28
- removed JP1, JP2, JP3: (no value), jumper:JP2
- removed Q7, Q8: BC847BS, transistor-small-signal:SOT363_PHILIPS
- removed R22, R23, R24, R44, R45, R46, R73, R74, R80: 1k, rcl:R0805
- removed R50, R57, R60, R64: 2k, rcl:R0805
- removed R54: 470R, rcl:R0805
- removed R55, R58, R61: 300, rcl:R0805
- removed R59, R62, R63: 30k, rcl:R0805
- removed R66, R71, R72: 12k, rcl:R0805
- removed RN5: 5, resistor-dil:EXB38V
- removed X2: (no value), con-ptr500:AK500/3
- added C33: 100nF, C_EU_Kando:C0603K
- added C34, C35: 4,7uF, C_EU_Kando:C0603K
- added D4: ll4148, Diodes:MINIMELF
- added D5: 40V, Diodes:MINIMELF
- added JP4: (no value), CONNECTORS:1X02
- added JP_CURRENT: (no value), CONNECTORS:1X04
- added L1: 4,7uH, Coils_Kando:WE-TPC_3816
- added MIC4607: MIC4607-1, MCHP_Egyeb_Kando:TSSOP28
- added MOTOR, X4: CLL5.08/3, CONNECTORS:CLL5.08/3
- added OBSRV1, OBSRV2, OBSRV3: (no value), CONNECTORS:1X03
- added R12: 22k 1%, R_EU:R0603
- added R13, R28: 0R, R_EU:R0603
- added R29, R30: 10R, R_EU:R0603
- added R34: 2,2k, R_EU:EXBV8V_A
- added R5: 68k 1%, R_EU:R0603
- added R6: 12k 1%, R_EU:R0603
- added T1, T2, T3: BSS123, Felvezetok:SOT23
- added U$1: MIC5233YM5, MCHP_Egyeb_Kando:TSOT23-5
- added U$2: MCP16301T-E/CH, MCHP_Egyeb_Kando:SOT23-6
- added X3: CLL5.08/2, CONNECTORS:CLL5.08/2
- 24V, 3.3V, 5V, 8V: value (none) -> Green; device led:CHIPLED_0805 -> Diodes:CHIPLED_0805
- ATA6563: value (none) -> ATA6563; device resistor-bourns:SO8 -> MCHP_Egyeb_Kando:SOIC-8
- C1, C2, C3: value 10u 16V -> 10uF; device rcl:C0805 -> C_EU_Kando:C0805K
- C12, C21, C22: value 47n -> 22nF; device rcl:C0805 -> C_EU_Kando:C0603K
- C13, C14, C15: value 56p -> 1nF; device rcl:C0805 -> C_EU_Kando:C0603K
- C16, C17, C18, C7: value 1n -> 1nF; device rcl:C0805 -> C_EU_Kando:C0603K
- C19: value 100n -> 1uF; device rcl:C0805 -> C_EU_Kando:C0603K
- C20: value 1n -> 22nF; device rcl:C0805 -> C_EU_Kando:C0603K
- C25, C29, C5: value 1u 50V -> 100nF; device rcl:C0805 -> C_EU_Kando:C0603K
- C26: value 1u 50V -> 1uF; device rcl:C0805 -> C_EU_Kando:C0603K
- C27, C28: value 100n -> 100nF; device rcl:C0805 -> C_EU_Kando:C0603K
- C31: value 2,2u 25V - ceramic -> 4,7uF; device rcl:C0805 -> C_EU_Kando:C0603K
- C32: value 4.7n -> 22nF; device rcl:C0805 -> C_EU_Kando:C0603K
- C4: value 1u 50V -> 22pF; device rcl:C0805 -> C_EU_Kando:C0603K
- C6: value 1u 50V -> 10uF; device rcl:C0805 -> C_EU_Kando:C1206
- C8: device rcl:TT5D10 -> C_EU_Kando:PANASONIC_E
- D1, D2, D3: value SD103BW -> 40V; device diode:SOD123 -> Diodes:MINIMELF
- EXT_SUPPLY: value (none) -> CLL5.08/2; device con-ptr500:AK500/2 -> CONNECTORS:CLL5.08/2
- FLT/EN_TP: device pinhead:1X02 -> CONNECTORS:1X03
- GND: device pinhead:1X01 -> CONNECTORS:1X02
- LED1, LED2, LED3, LED4, LED5, LED6: value (none) -> Yellow; device led:CHIPLED_0805 -> Diodes:CHIPLED_0805
- LED7, LED8: value (none) -> Red; device led:CHIPLED_0805 -> Diodes:CHIPLED_0805
- MCP6024: value (none) -> MCP6004ST; device MIC6024:SO14 -> MCHP_Egyeb_Kando:TSSOP14
- PWM_TEST_POINTS: device pinhead:1X06 -> CONNECTORS:1X06
- Q1, Q2, Q3, Q4, Q5, Q6: device transistor-power:PG-TDSON-8 -> Felvezetok:PG-TDSON-8_
- R1, R2, R3: value 3R -> 10R; device rcl:R0805 -> R_EU:R0603
- R10: value 30k -> 2,2k; device rcl:R0805 -> R_EU:EXBV8V_A
- R11: device rcl:R0805 -> R_EU:R0603
- R14, R21, R69: value 470R -> 680R; device rcl:R0805 -> R_EU:R0603
- R15, R17, R18: value 4.7k -> 2,2k; device rcl:R0805 -> R_EU:EXBV8V_A
- R16: value 4.7k -> 200R; device rcl:R0805 -> R_EU:EXBV8V_A
- R19: value 4.7k -> 22k; device rcl:R0805 -> R_EU:EXBV8V_A
- R20: value 4.7k -> 680R; device rcl:R0805 -> R_EU:R0603
- R25: value 56k -> 68k 1%; device rcl:R0805 -> R_EU:R0603
- R26, R27: device rcl:R0805 -> R_EU:R1206
- R4: value 5R -> 10R; device rcl:R0805 -> R_EU:R0603
- R47, R48: value 1k -> 2,2k; device rcl:R0805 -> R_EU:R0603
- R49, R51, R52, R77, R78, R79: value 33k -> 22k 1%; device rcl:R0805 -> R_EU:R0603
- R53, R56, R7, R75, R76, R9: value 0.01R -> R-EU_SMDR2512; device rcl:R2512 -> R_EU:R2512
- R65: value 10k -> 12k 1%; device rcl:R0805 -> R_EU:R0603
- R67: value 6k8 -> 12,4k 1%; device rcl:R0805 -> R_EU:R0603
- R68: value 2k2 -> 2,2k; device rcl:R0805 -> R_EU:R0603
- R70: value 470R -> 330R; device rcl:R0805 -> R_EU:R0603
- R8: value 499 -> 680R; device rcl:R0805 -> R_EU:R0603
- RN1, RN3, RN4: value 1k -> 2,2k; device resistor-dil:EXB38V -> R_EU:EXBV8V_A
- RN11, RN2: value 1k -> 680R; device resistor-dil:EXB38V -> R_EU:EXBV8V_A
- X1: value (none) -> CLL5.08/2; device con-phoenix-350_own:1751293 -> CONNECTORS:CLL5.08/2
- moved GND 82.6 mm to (3.81, 53.3), turned to 180 degrees
- moved C4 76.9 mm to (7.62, 22.9), turned to 0 degrees
- moved R65 56.5 mm to (59.7, 45.7), turned to 0 degrees
- moved EXT_SUPPLY 54.6 mm to (82.5, 7.62), turned to 180 degrees
- moved R25 54.5 mm to (59.7, 47.0)
- moved R17 51.2 mm to (24.1, 35.6), turned to 90 degrees
- moved 3.3V 50.7 mm to (46.4, 54.6), turned to 0 degrees
- moved C31 49.5 mm to (59.7, 40.6), turned to 0 degrees
- moved C6 48.7 mm to (85.1, 14.0), turned to 180 degrees
- moved C5 46.6 mm to (85.1, 16.5), turned to 180 degrees
- moved R70 45.3 mm to (46.4, 51.4), turned to 270 degrees
- moved R20 43.6 mm to (47.0, 19.1), turned to 180 degrees
- moved C26 43.2 mm to (53.3, 57.1), turned to 180 degrees
- moved R27 42.4 mm to (10.2, 17.8), turned to 180 degrees
- moved R67 41.8 mm to (44.5, 51.4), turned to 270 degrees
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Connections:
- removed net N$41: LED4.A, RN2.5
- removed net N$42: LED5.A, RN11.7
- removed net N$43: LED6.A, RN11.5
- removed net N$46: Q7.4, R74.1
- removed net N$50: Q8.1, R80.1
- removed net N$51: C12.1, R10.1, R57.2, R58.2
- removed net N$53: C22.1, R60.2, R61.2, R62.1
- new net N$12: C33.2, D5.C, L1.1, U$2.6
- new net N$44: R5.1, R6.1, U$2.3
- new net N$52: C33.1, D4.C, U$2.1
- new net N$56: C32.2, R26.2, R27.2
- net +24V: now also R19.5, U$1.1, U$1.3, U$2.4, U$2.5; no longer 1790.1, 5233.1, 5233.3, C4.1, R63.2
- net +5V: now also C34.1, C35.1, D4.A, L1.2, R34.6, R34.7, R34.8, R5.2, X3.1; no longer 1790.3, C23.1, R18.2, R19.2, R20.2, X1.2
- net +8V: now also MIC4607.21, U$1.5; no longer 5233.5, IC3.21
- net AHB: now also MIC4607.20; no longer IC3.20
- net AHO: now also MIC4607.19, R28.1; no longer IC3.19, RN5.2
- net AHS: now also MIC4607.18; no longer IC3.18
- net ALO: now also MIC4607.17, R30.2; no longer IC3.17, RN5.1
- net BHB: now also MIC4607.10; no longer IC3.10
- net BHO: now also MIC4607.11; no longer IC3.11
- net BHS: now also MIC4607.12; no longer IC3.12
- net BLO: now also MIC4607.13; no longer IC3.13
- net CAN_H: now also C4.1, X1.2; no longer C32.2, R26.2, R27.2, X1.6
- net CAN_L: now also C4.2, X1.1; no longer X1.7
- net CHB: now also MIC4607.27; no longer IC3.27
- net CHO: now also MIC4607.26, R13.1; no longer IC3.26, RN5.4
- net CHS: now also MIC4607.25; no longer IC3.25
- net CLO: now also MIC4607.24, R29.2; no longer IC3.24, RN5.3
- net DC_BUS: now also JP4.1, R17.5, R19.4; no longer DC_BUS_TP.1, R63.1, R64.2
- net EN: now also LED8.A, MIC4607.8; no longer IC3.8, R21.2
- net FLT: now also LED7.A, MIC4607.9, R12.1; no longer IC3.9, R14.2, R54.1
- net GND: now also C34.2, C35.2, D5.A, FLT/EN_TP.3, GND.2, JP4.2, JP_CURRENT.4, MIC4607.14, MIC4607.15, MIC4607.23, R14.1, R15.1, R15.2, R15.3, R17.1, R17.2, R17.3, R17.4, R20.2, R21.1, R6.2, U$1.2, U$2.2, X3.2; no longer 1790.2, 1790.4, 5233.2, C10.2, C11.2, C23.2, C30.2, C4.2, C9.2, IC3.1, IC3.14, IC3.15, IC3.23, IC3.28, LED7.C, LED8.C, R22.2, R23.2, R24.2, R50.1, R57.1, R60.1, R64.1, R73.2, R74.2, R80.2, X1.1
- net HALL_1/QEIA: now also R16.8; no longer Q7.6, R66.2
- net HALL_1/QEIA_IN: now also R34.1, X4.1; no longer R15.2, X1.3
- net HALL_2/QEIB: now also R16.6; no longer Q8.6, R72.2
- net HALL_2/QEIB_IN: now also R18.3, R34.3, X4.3; no longer R17.2, R20.1, X1.5
- net HALL_3/QEIINDEX: now also R16.7; no longer Q7.3, R71.2
- net HALL_3/QEIINDEX_IN: now also R18.2, R34.2, X4.2; no longer R16.2, R19.1, X1.4
- net ILIM+: now also MIC4607.16, R20.1; no longer IC3.16
- net N$14: now also U$1.4; no longer 5233.4
- net N$15: now also MCP6024.12; no longer MCP6024.10
- net N$16: now also R15.6, R16.3, T3.2; no longer LEFT.11
- net N$17: now also R15.7, R16.2, T2.2; no longer LEFT.12
- net N$18: now also R15.8, R16.1, T1.2; no longer LEFT.13
- net N$19: now also R18.8, T1.1; no longer C9.1, Q7.2, R15.1, R22.1
- net N$20: now also R18.7, T2.1; no longer C10.1, Q7.5, R16.1, R23.1
- net N$21: now also R13.2; no longer RN5.5
- net N$22: now also R28.2; no longer RN5.7
- net N$23: now also R18.6, T3.1; no longer C11.1, Q8.2, R17.1, R24.1
- net N$24: now also LED4.A, RN2.8; no longer C21.1, R50.2, R55.2, R59.1
- net N$25: now also LED3.A, RN2.7; no longer IC3.22
- net N$26: now also LED2.A, RN2.6; no longer LED1.A, RN2.8
- net N$3: now also MCP6024.14, R10.3; no longer MCP6024.8, R46.1
- net N$32: now also R29.1; no longer RN5.6
- net N$36: now also LED1.A, RN2.5; no longer Q7.1, R73.1
- net N$39: now also LED5.A, RN11.5; no longer LED2.A, RN2.7
- net N$4: now also R10.2; no longer R45.1
- net N$40: now also LED6.A, RN11.7; no longer LED3.A, RN2.6
- net N$49: now also MCP6024.13; no longer MCP6024.9
- net N$58: now also R30.1; no longer RN5.8
- net N$6: now also LED8.C, R21.2; no longer LED7.A, R14.1
- net N$60: now also R10.1; no longer R44.1
- net N$66: now also MCP6024.10; no longer MCP6024.12
- net N$8: now also LED7.C, R14.2; no longer LED8.A, R21.1
- net PHASE_CUR_1: now also JP_CURRENT.1, OBSRV1.1, R10.8; no longer JP1.1, P_CUR_1_TP.1, R44.2
- net PHASE_CUR_2: now also JP_CURRENT.2, OBSRV2.1, R10.7; no longer JP2.1, P_CUR_2_TP.1, R45.2
- net PHASE_CUR_SUM: now also JP_CURRENT.3, OBSRV3.1, R10.6; no longer JP3.1, P_CUR_SUM_TP.1, R46.2
- net PHASE_I_V_1: now also OBSRV1.2; no longer JP1.2
- net PHASE_I_V_2: now also OBSRV2.2; no longer JP2.2
- net PHASE_I_V_3: now also OBSRV3.2; no longer JP3.2
- net PHASE_VOLT_1: now also C12.1, OBSRV1.3, R17.8, R19.8; no longer JP1.3, R58.1
- net PHASE_VOLT_2: now also C21.1, OBSRV2.3, R17.7, R19.7; no longer JP2.3, R55.1
- net PHASE_VOLT_3: now also C22.1, OBSRV3.3, R17.6, R19.6; no longer JP3.3, R61.1
- net PWM1_H: now also MIC4607.7, RN2.3; no longer IC3.7, RN2.2
- net PWM1_L: now also MIC4607.6, RN2.4; no longer IC3.6, RN2.1
- net PWM2_H: now also MIC4607.5, RN2.1; no longer IC3.5, RN2.4
- net PWM2_L: now also MIC4607.4, RN2.2; no longer IC3.4, RN2.3
- net PWM3_H: now also MIC4607.3, RN11.2; no longer IC3.3, RN11.4
- net PWM3_L: now also MIC4607.2, RN11.4; no longer IC3.2, RN11.2
- net P_A: now also MOTOR.1, R19.1; no longer R10.2, X2.1
- net P_B: now also MOTOR.3, R19.2; no longer R59.2, X2.3
- net P_C: now also MOTOR.2, R19.3; no longer R62.2, X2.2
- net VDD: now also R12.2, T1.3, T2.3, T3.3; no longer C30.1, R54.2, R66.1, R71.1, R72.1
- net VREF: now also MCP6024.8, MCP6024.9; no longer MCP6024.13, MCP6024.14
Routing:
- net +5V: track 30.4 -> 172.1 mm, vias 0 -> 5
- net GND: track 524.6 -> 424.8 mm, vias 1 -> 18
- net SHUNT_HIGH_1: track 149.0 -> 78.3 mm
- net +24V: track 231.2 -> 164.0 mm, vias 0 -> 5
- net ILIM+: track 69.3 -> 11.8 mm, vias 2 -> 0
- net +8V: track 24.5 -> 76.6 mm, vias 0 -> 7
- net N$3: track 3.36 -> 50.5 mm, vias 0 -> 5
- net VDD: track 131.6 -> 177.4 mm, vias 3 -> 9
- net HALL_3/QEIINDEX: track 3.81 -> 40.5 mm, vias 0 -> 1
- net HALL_2/QEIB_IN: track 0.18 -> 34.4 mm, vias 0 -> 1
- net RXD_CAN: track 0.00 -> 33.9 mm, vias 0 -> 1
- net VREF: track 52.4 -> 18.7 mm
- net HALL_2/QEIB: track 2.54 -> 35.3 mm, vias 0 -> 1
- net PHASE_CUR_1: track 44.3 -> 76.6 mm, vias 1 -> 2
- net HALL_1/QEIA: track 1.27 -> 33.1 mm, vias 0 -> 1
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- added copper zone on layer 1, net GND
- added copper zone on layer 16, net GND
Other:
- board size 88.9 x 71.1 mm -> 88.9 x 59.7 mm
- board text added: "+"
- board text added: "A"
- board text added: "B"
- board text added: "C"
- board text added: "CANH CANL"
- board text added: "CURRENT"
- board text added: "DC"
- board text added: "EN FLT"
- board text added: "Hall/Encoder"
- board text added: "L1"
- board text added: "L2"
- board text added: "L3"
- board text added: "LED1-6"
- board text added: "MOTOR SHIELD REV.B"
- board text added: "OBSRV_1_2_3"
- board text added: "PWM"
- board text added: "UNIVERSAL"
- board text added: "VOLTAGE"
- board text added: "X2C"
- board text removed: "+8V"
- board text removed: "3,3V"
- board text removed: "DC_BUS VOLTAGE"
- board text removed: "EN"
- board text removed: "FLT"
- board text removed: "P.C.1"
- board text removed: "P.C.2"
- board text removed: "P.C.3"
- board text removed: "PWM1_H"
- board text removed: "PWM1_L"
- board text removed: "PWM2_H"
- board text removed: "PWM2_L"
- board text removed: "PWM3_1"
- board text removed: "PWM3_H"
- board text removed: "PWM3_L"
- board text removed: "P_A"
- board text removed: "P_B"
- board text removed: "P_C"
