File: MotorShield.sch (EAGLE design)
At the start: 141 parts, among them IC3 MIC4607, Q1 DMT4002LPS, Q2 DMT4002LPS, Q3 DMT4002LPS, Q4 DMT4002LPS, Q5 DMT4002LPS, Q6 DMT4002LPS, Q7 BC847BS, Q8 BC847BS, X1 1751293

Commit message: REVB version update
Parts:
- removed 1790: MCP1790-3302E/DB, Microchip_By_element14_Batch_1:MCP1790-3302E/DB
- removed 5233: MIC5233, MIC5233:MIC5233
- removed C10, C11, C9: 100p, rcl:C-EUC0805
- removed C23: 1u 50V, rcl:C-EUC0805
- removed C30: 100n, rcl:C-EUC0805
- removed DC_BUS_TP, P_CUR_1_TP, P_CUR_2_TP, P_CUR_SUM_TP: (no value), pinhead:PINHD-1X1
- removed IC3: MIC4607, daniic:ADUC814ARU
- removed JP1, JP2, JP3: (no value), jumper:JP2E
- removed Q7, Q8: BC847BS, transistor-small-signal:BC847BS
- removed R22, R23, R24, R44, R45, R46, R73, R74, R80: 1k, rcl:R-EU_R0805
- removed R50, R57, R60, R64: 2k, rcl:R-EU_R0805
- removed R54: 470R, rcl:R-EU_R0805
- removed R55, R58, R61: 300, rcl:R-EU_R0805
- removed R59, R62, R63: 30k, rcl:R-EU_R0805
- removed R66, R71, R72: 12k, rcl:R-EU_R0805
- removed RN5: 5, resistor-dil:4R-NEXB38V
- removed X2: (no value), con-ptr500:AK500/3
- added C33: 100nF, C_EU_Kando:C-EU-SMD_0603_100NF_50V
- added C34, C35: 4,7uF, C_EU_Kando:C-EU-SMD_0603_4,7UF_16V
- added D4: ll4148, Diodes:1N4148MINIMELF
- added D5: 40V, Diodes:SCHOTTKY40V
- added JP4: (no value), CONNECTORS:PINHD-1X2
- added JP_CURRENT: (no value), CONNECTORS:PINHD-1X4
- added L1: 4,7uH, Coils_Kando:WE-TPC_3816_4,7UH_0,9A
- added MIC4607: MIC4607-1, MCHP_Egyeb_Kando:MIC4607-1
- added MOTOR, X4: CLL5.08/3, CONNECTORS:AK500/3CSAVAROS_CLL5.08/3
- added OBSRV1, OBSRV2, OBSRV3: (no value), CONNECTORS:PINHD-1X3
- added R12: 22k 1%, R_EU:R-EU_SMDR0603_22K_1%
- added R13, R28: 0R, R_EU:R-EU_SMDR0603_0R
- added R29, R30: 10R, R_EU:R-EU_SMDR0603_3R
- added R34: 2,2k, R_EU:4R-N2,2K
- added R5: 68k 1%, R_EU:R-EU_SMDR0603_68K_1%
- added R6: 12k 1%, R_EU:R-EU_SMDR0603_12K_1%
- added T1, T2, T3: BSS123, Felvezetok:BSS123
- added U$1: MIC5233YM5, MCHP_Egyeb_Kando:MIC5233YM5
- added U$2: MCP16301T-E/CH, MCHP_Egyeb_Kando:MCP16301T-E/CH
- added X3: CLL5.08/2, CONNECTORS:AK500/2CSAVAROS_CLL5.08/2
- 24V, 3.3V, 5V, 8V: value (none) -> Green; device led:LEDCHIPLED_0805 -> Diodes:LEDCHIPLED_0805_GREEN
- ATA6563: value (none) -> ATA6563; device resistor-bourns:2NBS08-7 -> MCHP_Egyeb_Kando:ATA6563
- C1, C2, C3: value 10u 16V -> 10uF; device rcl:C-EUC0805 -> C_EU_Kando:C-EU-SMD_0805_10UF_16V
- C12, C21, C22: value 47n -> 22nF; device rcl:C-EUC0805 -> C_EU_Kando:C-EU-SMD_0603_22NF_16V
- C13, C14, C15: value 56p -> 1nF; device rcl:C-EUC0805 -> C_EU_Kando:C-EU-SMD_0603_1NF_100V
- C16, C17, C18, C7: value 1n -> 1nF; device rcl:C-EUC0805 -> C_EU_Kando:C-EU-SMD_0603_1NF_100V
- C19: value 100n -> 1uF; device rcl:C-EUC0805 -> C_EU_Kando:C-EU-SMD_0603_1UF_10V
- C20: value 1n -> 22nF; device rcl:C-EUC0805 -> C_EU_Kando:C-EU-SMD_0603_22NF_16V
- C25, C29, C5: value 1u 50V -> 100nF; device rcl:C-EUC0805 -> C_EU_Kando:C-EU-SMD_0603_100NF_50V
- C26: value 1u 50V -> 1uF; device rcl:C-EUC0805 -> C_EU_Kando:C-EU-SMD_0603_1UF_10V
- C27, C28: value 100n -> 100nF; device rcl:C-EUC0805 -> C_EU_Kando:C-EU-SMD_0603_100NF_50V
- C31: value 2,2u 25V - ceramic -> 4,7uF; device rcl:C-EUC0805 -> C_EU_Kando:C-EU-SMD_0603_4,7UF_16V
- C32: value 4.7n -> 22nF; device rcl:C-EUC0805 -> C_EU_Kando:C-EU-SMD_0603_22NF_16V
- C4: value 1u 50V -> 22pF; device rcl:C-EUC0805 -> C_EU_Kando:C-EU-SMD_0603_22PF_50V
- C6: value 1u 50V -> 10uF; device rcl:C-EUC0805 -> C_EU_Kando:C-EU-SMD_1206_10UF_50V
- C8: device rcl:CPOL-EUTT5D10 -> C_EU_Kando:CPOL-EUE
- D1, D2, D3: value SD103BW -> 40V; device diode:SD103BW -> Diodes:SCHOTTKY40V
- EXT_SUPPLY: value (none) -> CLL5.08/2; device con-ptr500:AK500/2 -> CONNECTORS:AK500/2CSAVAROS_CLL5.08/2
- FLT/EN_TP: device pinhead:PINHD-1X2 -> CONNECTORS:PINHD-1X3
- GND: device pinhead:PINHD-1X1 -> CONNECTORS:PINHD-1X2
- LED1, LED2, LED3, LED4, LED5, LED6: value (none) -> Yellow; device led:LEDCHIPLED_0805 -> Diodes:LEDCHIPLED_0805_YELLOW
- LED7, LED8: value (none) -> Red; device led:LEDCHIPLED_0805 -> Diodes:LEDCHIPLED_0805_RED
- MCP6024: value (none) -> MCP6004ST; device MIC6024:4AMP_P3+12D -> MCHP_Egyeb_Kando:MCP6004ST
- PWM_TEST_POINTS: device pinhead:PINHD-1X6 -> CONNECTORS:PINHD-1X6
- Q1, Q2, Q3, Q4, Q5, Q6: device transistor-power:BSZ105N04NS -> Felvezetok:BSZ105N04NS_PG-TDSON-8
- R1, R2, R3: value 3R -> 10R; device rcl:R-EU_R0805 -> R_EU:R-EU_SMDR0603_3R
- R10: value 30k -> 2,2k; device rcl:R-EU_R0805 -> R_EU:4R-N2,2K
- R11: device rcl:R-EU_R0805 -> R_EU:R-EU_SMDR0603_0R
- R14, R21, R69: value 470R -> 680R; device rcl:R-EU_R0805 -> R_EU:R-EU_SMDR0603_680R
- R15, R17, R18: value 4.7k -> 2,2k; device rcl:R-EU_R0805 -> R_EU:4R-N2,2K
- R16: value 4.7k -> 200R; device rcl:R-EU_R0805 -> R_EU:4R-N200R
- R19: value 4.7k -> 22k; device rcl:R-EU_R0805 -> R_EU:4R-N22K
- R20: value 4.7k -> 680R; device rcl:R-EU_R0805 -> R_EU:R-EU_SMDR0603_680R
- R25: value 56k -> 68k 1%; device rcl:R-EU_R0805 -> R_EU:R-EU_SMDR0603_68K_1%
- R26, R27: device rcl:R-EU_R0805 -> R_EU:R-EU_SMDR1206_60R
- R4: value 5R -> 10R; device rcl:R-EU_R0805 -> R_EU:R-EU_SMDR0603_3R
- R47, R48: value 1k -> 2,2k; device rcl:R-EU_R0805 -> R_EU:R-EU_SMDR0603_2,2K
- R49, R51, R52, R77, R78, R79: value 33k -> 22k 1%; device rcl:R-EU_R0805 -> R_EU:R-EU_SMDR0603_22K_1%
- R53, R56, R7, R75, R76, R9: value 0.01R -> R-EU_SMDR2512; device rcl:R-EU_R2512 -> R_EU:R-EU_SMDR2512
- R65: value 10k -> 12k 1%; device rcl:R-EU_R0805 -> R_EU:R-EU_SMDR0603_12K_1%
- R67: value 6k8 -> 12,4k 1%; device rcl:R-EU_R0805 -> R_EU:R-EU_SMDR0603_12,4K_1%
- R68: value 2k2 -> 2,2k; device rcl:R-EU_R0805 -> R_EU:R-EU_SMDR0603_2,2K
- R70: value 470R -> 330R; device rcl:R-EU_R0805 -> R_EU:R-EU_SMDR0603_330R
- R8: value 499 -> 680R; device rcl:R-EU_R0805 -> R_EU:R-EU_SMDR0603_680R
- RN1, RN3, RN4: value 1k -> 2,2k; device resistor-dil:4R-NEXB38V -> R_EU:4R-N2,2K
- RN11, RN2: value 1k -> 680R; device resistor-dil:4R-NEXB38V -> R_EU:4R-N680R
- X1: value 1751293 -> CLL5.08/2; device con-phoenix-350_own:1751293 -> CONNECTORS:AK500/2CSAVAROS_CLL5.08/2
Connections:
- removed net N$41: LED4.A, RN2D.2
- removed net N$42: LED5.A, RN11B.2
- removed net N$43: LED6.A, RN11D.2
- removed net N$46: Q7B.E1, R74.1
- removed net N$50: Q8A.E1, R80.1
- removed net N$51: C12.1, R10.1, R57.2, R58.2
- removed net N$53: C22.1, R60.2, R61.2, R62.1
- new net N$12: C33.2, D5.C, L1.1, U$2.SW
- new net N$44: R5.1, R6.1, U$2.VFB
- new net N$52: C33.1, D4.C, U$2.BOOST
- new net N$56: C32.2, R26.2, R27.2
- net +24V: now also R19D.2, U$1.EN, U$1.VIN, U$2.EN, U$2.VIN; no longer 1790.VIN, 5233.EN, 5233.IN, C4.1, R63.2
- net +5V: now also ATA6563.VCC, C34.1, C35.1, D4.A, L1.2, R34A.2, R34B.2, R34C.2, R5.2, X3-1.KL; no longer 1790.VOUT, ATA6563.3, C23.1, R18.2, R19.2, R20.2, X1-2.K
- net +8V: now also MIC4607.VDD, U$1.OUT; no longer 5233.OUT, IC3.VDD
- net AHB: now also MIC4607.AHB; no longer IC3.AHB
- net AHO: now also MIC4607.AHO, R28.1; no longer IC3.AHO, RN5B.1
- net AHS: now also MIC4607.AHS; no longer IC3.AHS
- net ALO: now also MIC4607.ALO, R30.2; no longer IC3.ALO, RN5A.1
- net BHB: now also MIC4607.BHB; no longer IC3.BHB
- net BHO: now also MIC4607.BHO; no longer IC3.BHO
- net BHS: now also MIC4607.BHS; no longer IC3.BHS
- net BLO: now also MIC4607.BLO; no longer IC3.BLO
- net CAN_H: now also ATA6563.CANH, C4.1, X1-2.KL; no longer ATA6563.7, C32.2, R26.2, R27.2, X1-6.K
- net CAN_L: now also ATA6563.CANL, C4.2, X1-1.KL; no longer ATA6563.6, X1-7.K
- net CHB: now also MIC4607.CHB; no longer IC3.CHB
- net CHO: now also MIC4607.CHO, R13.1; no longer IC3.CHO, RN5D.1
- net CHS: now also MIC4607.CHS; no longer IC3.CHS
- net CLO: now also MIC4607.CLO, R29.2; no longer IC3.CLO, RN5C.1
- net DC_BUS: now also JP4.1, R17D.2, R19D.1; no longer DC_BUS_TP.1, R63.1, R64.2
- net EN: now also LED8.A, MIC4607.EN; no longer IC3.EN, R21.2
- net FLT: now also LED7.A, MIC4607./FLT, R12.1; no longer IC3.FLT, R14.2, R54.1
- net GND: now also ATA6563.GND, ATA6563.STBY, C34.2, C35.2, D5.A, FLT/EN_TP.3, GND.2, JP4.2, JP_CURRENT.4, MIC4607.ILIM-, MIC4607.VSS, MIC4607.VSS2, R14.1, R15A.1, R15B.1, R15C.1, R17A.1, R17B.1, R17C.1, R17D.1, R20.2, R21.1, R6.2, U$1.GND, U$2.GND, X3-2.KL; no longer 1790.GND_(TAB), 1790.GND_(TAB)_2, 5233.GND, ATA6563.2, ATA6563.8, C10.2, C11.2, C23.2, C30.2, C4.2, C9.2, IC3.ILIM-, IC3.NC1, IC3.NC2, IC3.VSS, IC3.VSS1, LED7.C, LED8.C, R22.2, R23.2, R24.2, R50.1, R57.1, R60.1, R64.1, R73.2, R74.2, R80.2, X1-1.K
- net HALL_1/QEIA: now also R16A.2; no longer Q7A.C1, R66.2
- net HALL_1/QEIA_IN: now also R18A.1, R34A.1, X4-1.KL; no longer R15.2, R18.1, X1-3.K
- net HALL_2/QEIB: now also R16C.2; no longer Q8A.C1, R72.2
- net HALL_2/QEIB_IN: now also R18C.1, R34C.1, X4-3.KL; no longer R17.2, R20.1, X1-5.K
- net HALL_3/QEIINDEX: now also R16B.2; no longer Q7B.C1, R71.2
- net HALL_3/QEIINDEX_IN: now also R18B.1, R34B.1, X4-2.KL; no longer R16.2, R19.1, X1-4.K
- net ILIM+: now also MIC4607.ILIM+, R20.1; no longer IC3.ILIM+
- net N$14: now also U$1.ADJ; no longer 5233.ADJ.
- net N$16: now also R15C.2, R16C.1, T3.S; no longer LEFT.11
- net N$17: now also R15B.2, R16B.1, T2.S; no longer LEFT.12
- net N$18: now also R15A.2, R16A.1, T1.S; no longer LEFT.13
- net N$19: now also R18A.2, T1.G; no longer C9.1, Q7A.B1, R15.1, R22.1
- net N$20: now also R18B.2, T2.G; no longer C10.1, Q7B.B1, R16.1, R23.1
- net N$21: now also R13.2; no longer RN5D.2
- net N$22: now also R28.2; no longer RN5B.2
- net N$23: now also R18C.2, T3.G; no longer C11.1, Q8A.B1, R17.1, R24.1
- net N$24: now also LED4.A, RN2A.2; no longer C21.1, R50.2, R55.2, R59.1
- net N$25: now also LED3.A, RN2B.2; no longer IC3.DLY
- net N$26: now also LED2.A, RN2C.2; no longer LED1.A, RN2A.2
- net N$3: now also R10C.1; no longer R46.1
- net N$32: now also R29.1; no longer RN5C.2
- net N$36: now also LED1.A, RN2D.2; no longer Q7A.E1, R73.1
- net N$39: now also LED5.A, RN11D.2; no longer LED2.A, RN2B.2
- net N$4: now also R10B.1; no longer R45.1
- net N$40: now also LED6.A, RN11B.2; no longer LED3.A, RN2C.2
- net N$58: now also R30.1; no longer RN5A.2
- net N$6: now also LED8.C, R21.2; no longer LED7.A, R14.1
- net N$60: now also R10A.1; no longer R44.1
- net N$8: now also LED7.C, R14.2; no longer LED8.A, R21.1
- net PHASE_CUR_1: now also JP_CURRENT.1, OBSRV1.1, R10A.2; no longer JP1.1, P_CUR_1_TP.1, R44.2
- net PHASE_CUR_2: now also JP_CURRENT.2, OBSRV2.1, R10B.2; no longer JP2.1, P_CUR_2_TP.1, R45.2
- net PHASE_CUR_SUM: now also JP_CURRENT.3, OBSRV3.1, R10C.2; no longer JP3.1, P_CUR_SUM_TP.1, R46.2
- net PHASE_I_V_1: now also OBSRV1.2; no longer JP1.2
- net PHASE_I_V_2: now also OBSRV2.2; no longer JP2.2
- net PHASE_I_V_3: now also OBSRV3.2; no longer JP3.2
- net PHASE_VOLT_1: now also C12.1, OBSRV1.3, R17A.2, R19A.2; no longer JP1.3, R58.1
- net PHASE_VOLT_2: now also C21.1, OBSRV2.3, R17B.2, R19B.2; no longer JP2.3, R55.1
- net PHASE_VOLT_3: now also C22.1, OBSRV3.3, R17C.2, R19C.2; no longer JP3.3, R61.1
- net PWM1_H: now also MIC4607.AHI, RN2C.1; no longer IC3.AHI, RN2B.1
- net PWM1_L: now also MIC4607.ALI, RN2D.1; no longer IC3.ALI, RN2A.1
- net PWM2_H: now also MIC4607.BHI, RN2A.1; no longer IC3.BHI, RN2D.1
- net PWM2_L: now also MIC4607.BLI, RN2B.1; no longer IC3.BLI, RN2C.1
- net PWM3_H: now also MIC4607.CHI, RN11B.1; no longer IC3.CHI, RN11D.1
- net PWM3_L: now also MIC4607.CLI, RN11D.1; no longer IC3.CLI, RN11B.1
- net P_A: now also MOTOR-1.KL, R19A.1; no longer R10.2, X2-1.KL
- net P_B: now also MOTOR-3.KL, R19B.1; no longer R59.2, X2-3.KL
- net P_C: now also MOTOR-2.KL, R19C.1; no longer R62.2, X2-2.KL
- net RXD_CAN: now also ATA6563.RXD; no longer ATA6563.4
- net TXD_CAN: now also ATA6563.TXD; no longer ATA6563.1
- net VDD: now also ATA6563.VIO, R12.2, T1.D, T2.D, T3.D; no longer ATA6563.5, C30.1, R54.2, R66.1, R71.1, R72.1
